Commit message: added some files

File: limo_description/urdf/limo_four_diff.xacro (robot description, xacro)
@@ -26,5 +26,5 @@
             <origin xyz="0 0 -0.15" rpy="0 0 1.57" />
             <geometry>
-                <mesh filename="file://$(find limo_description)/meshes/limo_base.dae" scale="1 1 1"/>
+                <mesh filename="package://meshes/limo_base.dae" scale="1 1 1"/>
             </geometry>
         </visual>

File: limo_description/urdf/limo_four_diff_3dLidar.xacro (robot description, xacro)
@@ -150,20 +150,4 @@
     </sensor>
 </gazebo>
-  <!-- <joint name="base_joint" type="fixed">
-    <parent link="base_link"/>
-    <child link="velodyne_link"/>
-    <origin xyz="0.0 0.0 0.15" rpy="0 0 0"/>
-  </joint>
-  <link name="velodyne_link">
-  <visual name='base_footprint_fixed_joint_lump__velodyne_base_link_visual_1'>
-      <pose>0 0 -0.4 3.14159 0 3.14159</pose>
-      <geometry>
-          <mesh>
-              <scale>1 1 1</scale>
-              <uri>model://velodyne_description/meshes/VLP16_base_1.dae</uri>
-          </mesh>
-      </geometry>
-  </visual>
-  </link> -->
     <gazebo reference="front_left_wheel">
         <mu1>100</mu1>
@@ -201,8 +185,36 @@
         <fdir1>1 0 0</fdir1>
         <maxContacts value="64"/>
+    </gazebo>
+  <transmission name="right_wheel_trans">
+    <type>transmission_interface/SimpleTransmission</type>
+    <joint name="frobt_right_wheel">
+      <hardwareInterface>hardware_interface/VelocityJointInterface</hardwareInterface>
+    </joint>
+    <actuator name="right_wheel_motor">
+      <hardwareInterface>hardware_interface/VelocityJointInterface</hardwareInterface>
+      <mechanicalReduction>30</mechanicalReduction>
+    </actuator>
+  </transmission>
+  <transmission name="left_wheel_trans">
+    <type>transmission_interface/SimpleTransmission</type>
+    <joint name="front_left_wheel">
+      <hardwareInterface>hardware_interface/VelocityJointInterface</hardwareInterface>
+    </joint>
+    <actuator name="left_wheel_motor">
+      <hardwareInterface>hardware_interface/VelocityJointInterface</hardwareInterface>
+      <mechanicalReduction>30</mechanicalReduction>
+    </actuator>
+  </transmission>
+    <gazebo>
+      <plugin filename="libgazebo_ros_control.so" name="gazebo_ros_control"/>
     </gazebo>
     <gazebo>
         <plugin name="four_diff_controller" filename="libgazebo_ros_diff_drive.so">
-        <update_rate>50</update_rate>
+        <ros>
+            <namespace>/limo</namespace>
+            <!-- <argument>cmd_vel:=/cmd_vel</argument> -->
+            <!-- <argument>odom:=/odom</argument> -->
+			  </ros>
+        <update_rate>30</update_rate>
         <num_wheel_pairs>2</num_wheel_pairs>
         <left_joint>front_left_wheel</left_joint>
@@ -217,14 +229,24 @@
         <publish_odom>true</publish_odom>
         <publish_odom_tf>true</publish_odom_tf>
-        <publish_wheel_tf>true</publish_wheel_tf>
+        <publish_wheel_tf>false</publish_wheel_tf>
         <odometry_topic>odom</odometry_topic>
         <odometry_frame>odom</odometry_frame>
         <robot_base_frame>base_footprint</robot_base_frame>
-        <odometry_source>1</odometry_source>
-        <ros>
-            <remapping>odom:=/odometry</remapping>
-        </ros>
+        <!-- <odometry_source>1</odometry_source> -->
         </plugin>
     </gazebo>
+    <gazebo>
+    <plugin name="turtlebot3_joint_state" filename="libgazebo_ros_joint_state_publisher.so">
+      <ros>
+        <!-- <namespace>/tb3</namespace> -->
+        <remapping>~/out:=joint_states</remapping>
+      </ros>
+      <update_rate>30</update_rate>
+      <joint_name>front_left_wheel</joint_name>
+      <joint_name>front_right_wheel</joint_name>
+      <joint_name>rear_left_wheel</joint_name>
+      <joint_name>rear_right_wheel</joint_name>
+    </plugin>
+  </gazebo>
     <gazebo reference="velodyne_base_link" >
         <sensor name='velodyne-VLP16' type='ray'>

File: limo_description/urdf/limo_xacro.xacro (robot description, xacro)
@@ -11,5 +11,5 @@
                 <origin xyz="0 0 0" rpy="0 0 0" />
                 <geometry>
-                    <mesh filename="file://$(find limo_description)/meshes/limo_wheel.dae" />
+                    <mesh filename="package://meshes/limo_wheel.dae" />
                 </geometry>
             </visual>
