Commit message: updated some values for amcl

File: limo_description/urdf/limo_four_diff_3dLidar.xacro (robot description, xacro)
@@ -150,101 +150,45 @@
     </sensor>
 </gazebo>
-    <gazebo reference="front_left_wheel">
-        <mu1>100</mu1>
-        <mu2>100</mu2>
-        <kp>10000000.0</kp>
-        <kd>1.0</kd>
-        <minDepth>0.01</minDepth>
-        <fdir1>1 0 0</fdir1>
-        <maxContacts value="64"/>
-    </gazebo>
-    <gazebo reference="front_right_wheel">
-        <mu1>100</mu1>
-        <mu2>100</mu2>
-        <kp>10000000.0</kp>
-        <kd>1.0</kd>
-        <minDepth>0.01</minDepth>
-        <fdir1>1 0 0</fdir1>
-        <maxContacts value="64"/>
-    </gazebo>
-    <gazebo reference="rear_left_wheel">
-        <mu1>100</mu1>
-        <mu2>100</mu2>
-        <kp>10000000.0</kp>
-        <kd>1.0</kd>
-        <minDepth>0.01</minDepth>
-        <fdir1>1 0 0</fdir1>
-        <maxContacts value="64"/>
-    </gazebo>
-    <gazebo reference="rear_right_wheel">
-        <mu1>100</mu1>
-        <mu2>100</mu2>
-        <kp>10000000.0</kp>
-        <kd>1.0</kd>
-        <minDepth>0.01</minDepth>
-        <fdir1>1 0 0</fdir1>
-        <maxContacts value="64"/>
-    </gazebo>
-  <transmission name="right_wheel_trans">
-    <type>transmission_interface/SimpleTransmission</type>
-    <joint name="frobt_right_wheel">
-      <hardwareInterface>hardware_interface/VelocityJointInterface</hardwareInterface>
-    </joint>
-    <actuator name="right_wheel_motor">
-      <hardwareInterface>hardware_interface/VelocityJointInterface</hardwareInterface>
-      <mechanicalReduction>30</mechanicalReduction>
-    </actuator>
-  </transmission>
-  <transmission name="left_wheel_trans">
-    <type>transmission_interface/SimpleTransmission</type>
+    <ros2_control name="GazeboSystem" type="system">
+    <hardware>
+      <plugin>gazebo_ros2_control/GazeboSystem</plugin>
+    </hardware>
     <joint name="front_left_wheel">
-      <hardwareInterface>hardware_interface/VelocityJointInterface</hardwareInterface>
-    </joint>
-    <actuator name="left_wheel_motor">
-      <hardwareInterface>hardware_interface/VelocityJointInterface</hardwareInterface>
-      <mechanicalReduction>30</mechanicalReduction>
-    </actuator>
-  </transmission>
-    <gazebo>
-      <plugin filename="libgazebo_ros_control.so" name="gazebo_ros_control"/>
-    </gazebo>
-    <gazebo>
-        <plugin name="four_diff_controller" filename="libgazebo_ros_diff_drive.so">
-        <ros>
-            <namespace>/limo</namespace>
-            <!-- <argument>cmd_vel:=/cmd_vel</argument> -->
-            <!-- <argument>odom:=/odom</argument> -->
-			  </ros>
-        <update_rate>30</update_rate>
-        <num_wheel_pairs>2</num_wheel_pairs>
-        <left_joint>front_left_wheel</left_joint>
-        <right_joint>front_right_wheel</right_joint>
-        <left_joint>rear_left_wheel</left_joint>
-        <right_joint>rear_right_wheel</right_joint>
-        <wheel_separation>0.172</wheel_separation>
-        <wheel_diameter>0.09</wheel_diameter>
-        <max_wheel_torque>20</max_wheel_torque>
-        <max_wheel_acceleration>1.0</max_wheel_acceleration>
-        <command_topic>cmd_vel</command_topic>
-        <publish_odom>true</publish_odom>
-        <publish_odom_tf>true</publish_odom_tf>
-        <publish_wheel_tf>false</publish_wheel_tf>
-        <odometry_topic>odom</odometry_topic>
-        <odometry_frame>odom</odometry_frame>
-        <robot_base_frame>base_footprint</robot_base_frame>
-        <!-- <odometry_source>1</odometry_source> -->
-        </plugin>
-    </gazebo>
-    <gazebo>
-    <plugin name="turtlebot3_joint_state" filename="libgazebo_ros_joint_state_publisher.so">
-      <ros>
-        <!-- <namespace>/tb3</namespace> -->
-        <remapping>~/out:=joint_states</remapping>
-      </ros>
-      <update_rate>30</update_rate>
-      <joint_name>front_left_wheel</joint_name>
-      <joint_name>front_right_wheel</joint_name>
-      <joint_name>rear_left_wheel</joint_name>
-      <joint_name>rear_right_wheel</joint_name>
+      <command_interface name="velocity">
+        <param name="min">-1</param>
+        <param name="max">1</param>
+      </command_interface>
+      <state_interface name="position"/>
+      <state_interface name="velocity"/>
+    </joint>
+    <joint name="front_right_wheel">
+      <command_interface name="velocity">
+        <param name="min">-1</param>
+        <param name="max">1</param>
+      </command_interface>
+      <state_interface name="position"/>
+      <state_interface name="velocity"/>
+    </joint>
+    <joint name="rear_left_wheel">
+      <command_interface name="velocity">
+        <param name="min">-1</param>
+        <param name="max">1</param>
+      </command_interface>
+      <state_interface name="position"/>
+      <state_interface name="velocity"/>
+    </joint>
+    <joint name="rear_right_wheel">
+      <command_interface name="velocity">
+        <param name="min">-20</param>
+        <param name="max">20</param>
+      </command_interface>
+      <state_interface name="position"/>
+      <state_interface name="velocity"/>
+    </joint>
+    </ros2_control>
+  <gazebo>
+    <!-- Joint state publisher -->
+    <plugin filename="libgazebo_ros2_control.so" name="gazebo_ros2_control">
+      <parameters>$(find limo_description)/config/diff_drive_controller.yaml</parameters>
     </plugin>
   </gazebo>

File: limo_description/urdf/limo_xacro_3d.xacro (robot description, xacro)
@@ -5,6 +5,11 @@
             <inertial>
                 <origin xyz="0 0 0" />
-                <mass value="0.5" />
-                <inertia ixx="0.01055" ixy="0" ixz="0" iyy="0.00075" iyz="0" izz="0.01055" />
+                <mass value="2" />
+                <inertia ixx="0.145833"
+                        ixy="0.0"
+                        ixz="0.0"
+                        iyy="0.145833"
+                        iyz="0.0"
+                        izz="0.125"/>
             </inertial>
             <visual>

Commit message: added a new robot

File: limo_description/urdf/limo_four_diff_3dLidar.xacro (robot description, xacro)
@@ -180,6 +180,6 @@
     <joint name="rear_right_wheel">
       <command_interface name="velocity">
-        <param name="min">-20</param>
-        <param name="max">20</param>
+        <param name="min">-1</param>
+        <param name="max">1</param>
       </command_interface>
       <state_interface name="position"/>

File: limo_description/urdf/limo_xacro_3d copy.xacro (robot description, xacro)
@@ -1,21 +1,16 @@
 <?xml version="1.0"?>
 <robot name="limo_xacro" xmlns:xacro="http://ros.org/wiki/xacro">
-    <xacro:include filename="inertial_macros.xacro"/>
     <xacro:macro name="limo_wheel" params="parent_prefix wheel_prefix reflect *joint_pose">
         <link name="${wheel_prefix}_wheel_link">
-            <!-- <inertial>
+            <inertial>
                 <origin xyz="0 0 0" />
                 <mass value="0.5" />
                 <inertia ixx="0.01055" ixy="0" ixz="0" iyy="0.00075" iyz="0" izz="0.01055" />
-            </inertial> -->
-            <xacro:inertial_cylinder mass="0.5" length="${wheel_length}" radius="${wheel_radius}">
-                 <origin xyz="0 0 0" rpy="0 0 0"/>
-            </xacro:inertial_cylinder>
+            </inertial>
             <visual>
-                <origin xyz="0 ${wheel_length/2} 0" rpy="1.57 0 0" />
+                <origin xyz="0 0 0" rpy="0 0 0" />
                 <geometry>
-                    <cylinder radius="${wheel_radius}" length="${wheel_length}"/>
+                    <mesh filename="file://$(find limo_description)/meshes/limo_wheel.dae" />
                 </geometry>
-                <!-- <material name="blue"/> -->
             </visual>
             <collision>
